File: sch/HX8357.sch (KiCad schematic (older format))
At the start: 40 parts, among them J1 BARREL_JACK, J2 CONN_01X02, J3 ICSP, J4 HX8357, Q1 MMBT2222A, U1 LM7805CV, U2 ATMEGA328P-PU, U3 DS1307, U4 PSW-8,5R, U5 MAX485CSA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

Commit message: Signed-off-by: cuki2 <mauricio@krebs.com.br>
Parts:
- U5: footprint Housings_SOIC:SOIC-8_3.9x4.9mm_Pitch1.27mm -> w_smd_dil:so-8; Equitronic (none) -> 7859; MNP (none) -> MAX485ESA+
Changed lines of the file:
@@
 F 0 "U5" H 9400 1950 50  0000 L CNN
 F 1 "MAX485CSA" H 9800 1950 50  0000 L CNN
-F 2 "Housings_SOIC:SOIC-8_3.9x4.9mm_Pitch1.27mm" H 10750 1250 50  0001 C CIN
-F 3 "" H 9700 1600 50  0001 C CNN
+F 2 "w_smd_dil:so-8" H 10750 1250 50  0001 C CIN
+F 3 "https://datasheets.maximintegrated.com/en/ds/MAX1487-MAX491.pdf" H 9700 1600 50  0001 C CNN
+F 4 "MAX485ESA+" H 9700 1600 60  0001 C CNN "MNP"
+F 5 "7859" H 9700 1600 60  0001 C CNN "Equitronic"
 	1    9700 1600
 	1    0    0    -1

Commit message: Signed-off-by: cuki2 <mauricio@krebs.com.br>
Parts:
- removed C10, C9: 22pF, w_smd_cap:c_0805, symbol C
- added R11, R12: 4k7, w_smd_resistors:r_0805, symbol R
Connections:
- net +5V: now also R11.2, R12.2
- net SCL: now also R12.1
- net SDA: now also R11.1
Other:
- moved on the sheet: BT1, Y2
