File: sch/HX8357.kicad_pcb (KiCad board)
At the start: 2 copper layers, 89.9 x 54.2 mm, 44 parts, among them J1 BARREL_JACK, J2 CONN_01X02, J3 ICSP, J4 HX8357, Q1 MMBT2222A, U1 LM7805CV, U2 ATMEGA328P-PU, U3 DS1307, U4 PSW-8,5R, U5 MAX485CSA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

Commit message: Placa
Signed-off-by: cuki2 <mauricio@krebs.com.br>
Routing:
- net /DB10: track 0.00 -> 90.3 mm, vias 0 -> 1
- net /DB11: track 0.00 -> 82.7 mm, vias 0 -> 2
- net /SCK: track 0.00 -> 78.7 mm, vias 0 -> 3
- net /WR: track 0.00 -> 76.4 mm, vias 0 -> 5
- net /DB12: track 0.00 -> 73.7 mm, vias 0 -> 4
- net /SD_CS: track 0.00 -> 72.4 mm, vias 0 -> 5
- net /DB13: track 0.00 -> 69.1 mm, vias 0 -> 2
- net /DB14: track 0.00 -> 62.8 mm, vias 0 -> 4
- net /DB15: track 0.00 -> 62.4 mm, vias 0 -> 3
- net /PB4: track 0.00 -> 59.0 mm, vias 0 -> 5
- net /PB3: track 0.00 -> 57.9 mm, vias 0 -> 5
- net /RS: track 0.00 -> 57.8 mm, vias 0 -> 1
- net +5V: track 239.3 -> 286.4 mm, vias 4 -> 5
- net /RST: track 0.00 -> 32.7 mm, vias 0 -> 2
- net GND: track 274.2 -> 304.5 mm, vias 7 -> 8
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
Commit message: Signed-off-by: cuki2 <mauricio@krebs.com.br>
Routing:
- net GND: track 304.5 -> 346.1 mm, vias 8 -> 13
Changed lines of the file:
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@@
     (thickness 1.6)
     (drawings 4)
-    (tracks 602)
+    (tracks 621)
     (zones 0)
     (modules 44)
@@
     (visible_elements 7FFFFF7F)
     (pcbplotparams
-      (layerselection 0x011fc_80000001)
+      (layerselection 0x010f0_80000001)
       (usegerberextensions false)
       (excludeedgelayer true)
@@
       (padsonsilk false)
       (subtractmaskfromsilk false)
-      (outputformat 4)
+      (outputformat 1)
       (mirror false)
       (drillshape 0)
       (scaleselection 1)
-      (outputdirectory pdf))
+      (outputdirectory gerber))
   )
   (net 0 "")
@@
   (gr_line (start 20 20) (end 20 74.25) (angle 90) (layer Edge.Cuts) (width 0.15))
   (gr_line (start 20 20) (end 109.92 20) (angle 90) (layer Edge.Cuts) (width 0.15))
+  (via (at 97.409 67.691) (size 0.6) (drill 0.4) (layers F.Cu B.Cu) (net 1))
+  (segment (start 97.409 67.691) (end 92.964 67.691) (width 0.4) (layer F.Cu) (net 1))
+  (segment (start 78.359 65.659) (end 74.549 61.849) (width 0.4) (layer B.Cu) (net 1))
+  (segment (start 74.549 61.849) (end 68.961 61.849) (width 0.4) (layer B.Cu) (net 1))
+  (via (at 68.961 61.849) (size 0.6) (drill 0.4) (layers F.Cu B.Cu) (net 1))
+  (via (at 78.359 67.31) (size 0.6) (drill 0.4) (layers F.Cu B.Cu) (net 1))
+  (segment (start 78.359 67.31) (end 78.359 65.659) (width 0.4) (layer B.Cu) (net 1))
+  (segment (start 78.359 67.31) (end 78.867 66.802) (width 0.4) (layer B.Cu) (net 1))
+  (segment (start 69.723 69.723) (end 70.231 69.215) (width 0.4) (layer B.Cu) (net 1))
+  (segment (start 70.231 69.215) (end 76.454 69.215) (width 0.4) (layer B.Cu) (net 1))
+  (segment (start 76.454 69.215) (end 78.359 67.31) (width 0.4) (layer B.Cu) (net 1))
+  (via (at 66.421 69.723) (size 0.6) (drill 0.4) (layers F.Cu B.Cu) (net 1))
+  (segment (start 60.198 68.961) (end 60.96 69.723) (width 0.4) (layer F.Cu) (net 1))
+  (segment (start 66.421 69.723) (end 60.96 69.723) (width 0.4) (layer F.Cu) (net 1))
+  (segment (start 60.198 67.31) (end 60.198 68.961) (width 0.4) (layer F.Cu) (net 1))
+  (segment (start 66.421 69.723) (end 69.723 69.723) (width 0.4) (layer B.Cu) (net 1))
+  (via (at 85.725 67.564) (size 0.6) (drill 0.4) (layers F.Cu B.Cu) (net 1))
+  (segment (start 84.963 66.802) (end 85.725 67.564) (width 0.4) (layer B.Cu) (net 1))
+  (segment (start 78.867 66.802) (end 84.963 66.802) (width 0.4) (layer B.Cu) (net 1))
   (segment (start 90.3605 61.976) (end 90.3605 60.5155) (width 0.4) (layer F.Cu) (net 1))
   (segment (start 88.519 57.531) (end 88.519 55.626) (width 0.4) (layer B.Cu) (net 1))
@@
   (segment (start 90.3605 65.0875) (end 90.3605 61.976) (width 0.4) (layer F.Cu) (net 1))
   (segment (start 92.964 67.691) (end 90.3605 65.0875) (width 0.4) (layer F.Cu) (net 1))
-  (segment (start 101.6 67.691) (end 92.964 67.691) (width 0.4) (layer F.Cu) (net 1))
+  (segment (start 101.6 67.691) (end 97.409 67.691) (width 0.4) (layer F.Cu) (net 1))
   (segment (start 102.624 68.715) (end 101.6 67.691) (width 0.4) (layer F.Cu) (net 1))
   (segment (start 108.4 68.715) (end 105.86 68.715) (width 0.4) (layer F.Cu) (net 1))
